Commit message: [fix] readme.md urdf2sdf conversion command [feature] camera image added added to rviz_config, camera plugin added to car_camera.xacro [test] tested on ros2 humble

File: car/car_camera/model.xacro (robot description, xacro)
@@ -34,3 +34,28 @@
         </visual>
     </link>
+    <gazebo reference="car_camera">
+        <sensor type="camera" name="car_camera">
+            <update_rate>24</update_rate>
+            <visualize>true</visualize>
+            <camera name="head">
+                <horizontal_fov>1.3962634</horizontal_fov>
+                <image>
+                    <width>640</width>
+                    <height>480</height>
+                    <format>R8G8B8</format>
+                </image>
+                <clip>
+                    <near>0.02</near>
+                    <far>300</far>
+                </clip>
+            </camera>
+            <plugin name="camera_controller" filename="libgazebo_ros_camera.so">
+                <ros>
+                    <!-- <namespace>camera</namespace> -->
+                    <argument>--ros-args --remap image_raw:=image_raw</argument>
+                    <argument>--ros-args --remap camera_info:=camera_info</argument>
+                </ros>
+            </plugin>
+        </sensor>
+    </gazebo>
 </robot>

File: car/model.urdf (robot description, URDF)
Before this commit: robot 2wheel_drive_car, 8 links, 7 joints
Links:
- removed link camera_ros
- added link car_camera, mass 0.1; collision box size=0.1 0.1 0.1; visual box size=0.1 0.1 0.1
Joints:
- joint camera_2_body: child camera_ros -> car_camera

File: car/model.xacro (robot description, xacro)
@@ -52,9 +52,9 @@
         <dynamics friction="0.5"/>
     </joint>
-    <xacro:include filename="camera_ros/model.xacro"/>
+    <xacro:include filename="car_camera/model.xacro"/>
     <joint name="camera_2_body" type="fixed">
         <origin xyz="${+(car_body_length/2) - (camera_length/2)} 0 ${car_body_height/2 + camera_length/2}" rpy="0 0 0"/>
         <parent link="car_body"/>
-        <child link="camera_ros"/>
+        <child link="car_camera"/>
     </joint>
     <gazebo>

Commit message: [feature][edit] xacro, urdf and sdf files modified to match ignition gazebo [test] urdf files tested with ros2 rivz (urdf_tutorial package) [test] sdf files tested with ign gazebo [test] bridge between ign gazebo and ros tested with ros_ign_gazebo parameter_bridge and ignition_gazebo_diff_drive_system plugin combined with ros2 teleop_twist_keyboard package

File: car/car_camera/model.xacro (robot description, xacro)
@@ -38,4 +38,5 @@
             <update_rate>24</update_rate>
             <visualize>true</visualize>
+            <topic>camera</topic>
             <camera name="head">
                 <horizontal_fov>1.3962634</horizontal_fov>
@@ -50,12 +51,30 @@
                 </clip>
             </camera>
-            <plugin name="camera_controller" filename="libgazebo_ros_camera.so">
-                <ros>
-                    <!-- <namespace>camera</namespace> -->
-                    <argument>--ros-args --remap image_raw:=image_raw</argument>
-                    <argument>--ros-args --remap camera_info:=camera_info</argument>
-                </ros>
+        </sensor>
+        <!-- <sensor type="camera" name="car_camera">
+            <update_rate>24</update_rate>
+            <visualize>true</visualize>
+            <camera name="head">
+                <horizontal_fov>1.3962634</horizontal_fov>
+                <image>
+                    <width>640</width>
+                    <height>480</height>
+                    <format>R8G8B8</format>
+                </image>
+                <clip>
+                    <near>0.02</near>
+                    <far>300</far>
+                </clip>
+            </camera>
+            <plugin filename="CameraTracking" name="Camera Tracking">
+                <ignition-gui>
+                    <property key="resizable" type="bool">false</property>
+                    <property key="width" type="double">5</property>
+                    <property key="height" type="double">5</property>
+                    <property key="state" type="string">floating</property>
+                    <property key="showTitleBar" type="bool">false</property>
+                </ignition-gui>
             </plugin>
-        </sensor>
+        </sensor> -->
     </gazebo>
 </robot>

File: car/car_wheel/model.xacro (robot description, xacro)
@@ -1,4 +1,4 @@
 <?xml version='1.0'?>
-<robot xmlns:xacro="http://www.ros.org/wiki/xacro" name="car_car_ball_wheel">
+<robot xmlns:xacro="http://www.ros.org/wiki/xacro" name="car_car_wheel">
     <xacro:property name="car_wheel_radius" value="0.25" />
     <xacro:property name="car_wheel_mass" value="0.5" />

File: car/model.xacro (robot description, xacro)
@@ -20,6 +20,5 @@
     <xacro:car_ball_wheel name="rear_right_ball_wheel"/>
     <joint name="rear_right_ball_wheel_2_body" type="continuous">
-        <origin xyz="${-(car_body_length/2) + (car_body_length/5)} ${-(car_body_width/2) + (car_body_width/5)} ${-(car_body_height/2)}"
-        rpy="0.0 0.0 0.0"/>
+        <origin xyz="${-(car_body_length/2) + (car_body_length/5)} ${-(car_body_width/2) + (car_body_width/5)} ${-(car_body_height/2)}" rpy="0.0 0.0 0.0"/>
         <parent link="car_body"/>
         <child link="rear_right_ball_wheel"/>
@@ -59,24 +58,31 @@
     </joint>
     <gazebo>
-        <plugin name="two_wheeled_robot_diff_drive" filename="libgazebo_ros_diff_drive.so">
-            <!-- Number of wheel pairs -->
-            <num_wheel_pairs>1</num_wheel_pairs>
-            <!-- wheels0 -->
+        <plugin filename="ignition-gazebo-diff-drive-system" name="ignition::gazebo::systems::DiffDrive">
             <left_joint>front_left_wheel_2_body</left_joint>
             <right_joint>front_right_wheel_2_body</right_joint>
-            <!-- kinematics -->
+            <wheel_separation>1</wheel_separation>
+            <wheel_radius>${car_wheel_radius}</wheel_radius>
+            <odom_publish_frequency>1</odom_publish_frequency>
+            <max_linear_acceleration>1</max_linear_acceleration>
+            <min_linear_acceleration>-1</min_linear_acceleration>
+            <max_angular_acceleration>2</max_angular_acceleration>
+            <min_angular_acceleration>-2</min_angular_acceleration>
+            <max_linear_velocity>0.5</max_linear_velocity>
+            <min_linear_velocity>-0.5</min_linear_velocity>
+            <max_angular_velocity>1</max_angular_velocity>
+            <min_angular_velocity>-1</min_angular_velocity>
+        </plugin>
+        <!-- <plugin name="two_wheeled_robot_diff_drive" filename="libgazebo_ros_diff_drive.so">
+            <num_wheel_pairs>1</num_wheel_pairs>
+            <left_joint>front_left_wheel_2_body</left_joint>
+            <right_joint>front_right_wheel_2_body</right_joint>
             <wheel_separation>1</wheel_separation>
             <wheel_diameter>0.5</wheel_diameter>
-            <!-- limits -->
             <max_wheel_torque>20</max_wheel_torque>
-            <!-- <max_wheel_acceleration>5.0</max_wheel_acceleration> -->
-            <!-- output -->
             <publish_odom>true</publish_odom>
             <publish_odom_tf>true</publish_odom_tf>
-            <!-- <publish_wheel_tf>true</publish_wheel_tf> -->
-            <!-- <ros><argument>cmd_vel:=custom_cmd_vel</argument></ros> -->
             <odometry_frame>start_loc_map</odometry_frame>
             <robot_base_frame>car_body::link</robot_base_frame>
-        </plugin>
+        </plugin> -->
     </gazebo>
 </robot>
