Commit message: [feature] joint_state_publisher plugin [edit] rviz & ign_gazebo config [edit] readme.md update [fix] tf tree and model description

File: car/model.urdf (robot description, URDF)
Before this commit: robot 2wheel_drive_car, 8 links, 7 joints
Links:
- removed link car_body::link
Joints:
- removed joint camera_2_body
- removed joint carbodylink_2_carbody
- removed joint front_left_wheel_2_body
- removed joint front_right_wheel_2_body
- removed joint rear_left_ball_wheel_2_body
- removed joint rear_right_ball_wheel_2_body
- added joint camera_to_body: type fixed, parent car_body, child car_camera, origin xyz=0.95 0 0.3 rpy=0 0 0
- added joint front_left_wheel_to_body: type continuous, parent car_body, child front_left_wheel, origin xyz=0.6 0.5 -0.125 rpy=-1.5707963267948966 0 0, axis 0 0 1
- added joint front_right_wheel_to_body: type continuous, parent car_body, child front_right_wheel, origin xyz=0.6 -0.5 -0.125 rpy=-1.5707963267948966 0 0, axis 0 0 1
- added joint rear_left_ball_wheel_to_body: type continuous, parent car_body, child rear_left_ball_wheel, origin xyz=-0.6 0.3 -0.25 rpy=0.0 0.0 0.0, axis 0 1 0
- added joint rear_right_ball_wheel_to_body: type continuous, parent car_body, child rear_right_ball_wheel, origin xyz=-0.6 -0.3 -0.25 rpy=0.0 0.0 0.0, axis 0 1 0
- joint base_link: child base_footprint -> car_body; origin xyz=0 0 -0.375 rpy=0 0 0 -> xyz=0 0 0.375 rpy=0 0 0; parent car_body -> base_footprint

File: car/model.xacro (robot description, xacro)
@@ -2,8 +2,8 @@
 <robot xmlns:xacro="http://www.ros.org/wiki/xacro" name="2wheel_drive_car">
     <!-- car body -->
-    <link name="car_body::link" />
+    <link name="car_body__link" />
     <xacro:include filename="car_body/model.xacro"/>
-    <joint name="carbodylink_2_carbody" type="fixed">
-        <parent link="car_body::link"/>
+    <joint name="carbodylink_to_carbody" type="fixed">
+        <parent link="car_body__link"/>
         <child link="car_body"/>
     </joint>
@@ -11,5 +11,5 @@
     <xacro:include filename="car_ball_wheel/model.xacro"/>
     <xacro:car_ball_wheel name="rear_left_ball_wheel"/>
-    <joint name="rear_left_ball_wheel_2_body" type="continuous">
+    <joint name="rear_left_ball_wheel_to_body" type="continuous">
         <origin xyz="${-(car_body_length/2) + (car_body_length/5)} ${(car_body_width/2) - (car_body_width/5)} ${-(car_body_height/2)}" rpy="0.0 0.0 0.0"/>
         <parent link="car_body"/>
@@ -19,5 +19,5 @@
     </joint>
     <xacro:car_ball_wheel name="rear_right_ball_wheel"/>
-    <joint name="rear_right_ball_wheel_2_body" type="continuous">
+    <joint name="rear_right_ball_wheel_to_body" type="continuous">
         <origin xyz="${-(car_body_length/2) + (car_body_length/5)} ${-(car_body_width/2) + (car_body_width/5)} ${-(car_body_height/2)}" rpy="0.0 0.0 0.0"/>
         <parent link="car_body"/>
@@ -36,5 +36,5 @@
     <xacro:include filename="car_wheel/model.xacro"/>
     <xacro:car_wheel name="front_left_wheel"/>
-    <joint name="front_left_wheel_2_body" type="continuous">
+    <joint name="front_left_wheel_to_body" type="continuous">
         <origin xyz="${+(car_body_length/2) - (car_body_length/5)} ${(car_body_width/2)} ${-(car_body_height/2) + (car_wheel_radius - car_ball_wheel_radius)}" rpy="${-pi/2} 0 0"/>
         <parent link="car_body"/>
@@ -44,5 +44,5 @@
     </joint>
     <xacro:car_wheel name="front_right_wheel"/>
-    <joint name="front_right_wheel_2_body" type="continuous">
+    <joint name="front_right_wheel_to_body" type="continuous">
         <origin xyz="${+(car_body_length/2) - (car_body_length/5)} ${-(car_body_width/2)} ${-(car_body_height/2) + (car_wheel_radius - car_ball_wheel_radius)}" rpy="${-pi/2} 0 0"/>
         <parent link="car_body"/>
@@ -52,5 +52,5 @@
     </joint>
     <xacro:include filename="car_camera/model.xacro"/>
-    <joint name="camera_2_body" type="fixed">
+    <joint name="camera_to_body" type="fixed">
         <origin xyz="${+(car_body_length/2) - (camera_length/2)} 0 ${car_body_height/2 + camera_length/2}" rpy="0 0 0"/>
         <parent link="car_body"/>
@@ -59,6 +59,10 @@
     <gazebo>
         <plugin filename="ignition-gazebo-diff-drive-system" name="ignition::gazebo::systems::DiffDrive">
-            <left_joint>front_left_wheel_2_body</left_joint>
-            <right_joint>front_right_wheel_2_body</right_joint>
+            <left_joint>front_left_wheel_to_body</left_joint>
+            <right_joint>front_right_wheel_to_body</right_joint>
+            <odom_topic>odometry</odom_topic>
+            <tf_topic>tf</tf_topic>
+            <frame_id>odom</frame_id>
+            <child_frame>car_body__link</child_frame>
             <wheel_separation>1</wheel_separation>
             <wheel_radius>${car_wheel_radius}</wheel_radius>
@@ -73,10 +77,6 @@
             <min_angular_velocity>-1</min_angular_velocity>
         </plugin>
-        <!-- <plugin filename="libignition-gazebo6-joint-state-publisher-system.so.6.9.0" name="ignition::gazebo::systems::JointStatePublisher ">
-            <joint_name>front_right_wheel</joint_name>
-            <joint_name>front_left_wheel</joint_name>
-            <joint_name>rear_right_ball_wheel</joint_name>
-            <joint_name>rear_left_ball_wheel</joint_name>
-        </plugin> -->
+        <plugin filename="libignition-gazebo-joint-state-publisher-system.so" name="ignition::gazebo::systems::JointStatePublisher ">
+        </plugin>
     </gazebo>
 </robot>
